File: Paddle/paddle.sch (EAGLE design)
At the start: 14 parts, among them U1 LMV321SEG-7SOT25, U2 MCP3221A5T-E/OT

Commit message: Added Copyright, License and Frame
Other:
- note added: "12bit Resolution, IIC Terminated"
- note added: "Amplifier and IIC Digitizer"
- note added: "Copyright (C) 2014 H.Poetzl Licensed under CERN OHL v.1.1"
- note added: "Paddle Controller"
- moved on the sheet: C1, C2, GND, P1, POT, R1, R2, SCL, SDA, U1, U2, VCC
